File: PoweUnit/PoweUnit.kicad_pcb (KiCad board)
At the start: 2 copper layers, 18 parts, among them J1 Jack-DC, J3 Conn_01x02, Q1 Q_PMOS_GDS, SW1 SW_Slide_DPDT, SW2 SW_SPST, U1 NE555D, U2 NJM2746M

Commit message: パワーパック完成
Parts:
- added C3: 0.1u, Capacitor_THT:C_Disc_D5.1mm_W3.2mm_P5.00mm, F.Cu at (146.5, 89.0)
- added G***: LOGO, LOGO, F.Cu at (115.5, 65.2)
- added J2: Conn_01x02_Pin, Connector_PinHeader_2.54mm:PinHeader_1x02_P2.54mm_Horizontal, F.Cu at (165.8, 112.5)
- added J4: Conn_01x02, Connector_JST:JST_XH_S2B-XH-A_1x02_P2.50mm_Horizontal, F.Cu at (135.0, 50.0)
- added R6: 10k, Resistor_THT:R_Axial_DIN0207_L6.3mm_D2.5mm_P7.62mm_Horizontal, F.Cu at (141.2, 80.0)
- added REF**: MountingHole_3.2mm_M3, MountingHole:MountingHole_3.2mm_M3, F.Cu at (105.0, 105.0)
- added REF**: MountingHole_3.2mm_M3, MountingHole:MountingHole_3.2mm_M3, F.Cu at (165.0, 105.0)
- added REF**: MountingHole_3.2mm_M3, MountingHole:MountingHole_3.2mm_M3, F.Cu at (105.0, 55.0)
- added REF**: MountingHole_3.2mm_M3, MountingHole:MountingHole_3.2mm_M3, F.Cu at (165.0, 55.0)
- D1: value short -> LED
- D2: value LED -> short
- J3: value Conn_01x02 -> Conn_01x02_Socket; footprint Connector_JST:JST_XH_S2B-XH-A_1x02_P2.50mm_Horizontal -> Connector_PinSocket_2.54mm:PinSocket_1x02_P2.54mm_Horizontal
- R2: value 1.2k -> 5.1k
- R3: value 3k -> 1.2k
- R4: value 10k -> 3k
- SW1: value SW_Slide_DPDT -> SW_SPST; footprint samacsys:SS22F06G5G -> MyLibrary:CW-SB11KKFF
- SW2: value SW_SPST -> SW_Slide_DPDT; footprint MyLibrary:CW-SB11KKFF -> samacsys:SS22F06G5G
- moved C1 65.8 mm to (127.7, 82.7), turned to -90 degrees
- moved C2 59.9 mm to (127.8, 96.2)
- moved J3 59.2 mm to (110.5, 112.5)
- moved Q1 55.5 mm to (142.7, 83.2)
- moved SW2 54.3 mm to (135.0, 77.0), turned to 90 degrees
- moved U1 46.1 mm to (130.2, 91.5), turned to 180 degrees
- moved U2 45.5 mm to (140.2, 91.5)
- moved D2 43.7 mm to (131.8, 103.0), turned to -90 degrees
- moved R5 41.7 mm to (148.8, 86.2), turned to 180 degrees
- moved R4 40.6 mm to (124.2, 90.2), turned to 90 degrees
- moved J1 38.5 mm to (118.8, 120.0), turned to 90 degrees
- moved F1 37.6 mm to (125.2, 112.5), turned to 90 degrees
- moved RV1 35.3 mm to (156.5, 85.0), turned to 90 degrees
- moved D1 31.8 mm to (131.8, 113.0), turned to -90 degrees
- moved SW1 31.0 mm to (113.5, 90.0), turned to 180 degrees
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Connections:
- C2 pad 1: Net-(Q1-S) -> VCC
- F1 pad 2: Net-(SW2-A) -> Net-(SW1-A)
- J3 pad 1: /Feeder+ -> +12V
- J3 pad 2: /Feeder- -> GND
- Q1 pad 3: Net-(Q1-S) -> VCC
- R1 pad 1: Net-(SW2-A) -> Net-(D1-K)
- R1 pad 2: Net-(D1-K) -> GND
- R2 pad 1: Net-(Q1-S) -> Net-(SW1-A)
- R2 pad 2: Net-(U1-DISCH) -> Net-(D2-K)
- R3 pad 1: Net-(U1-DISCH) -> VCC
- R3 pad 2: Net-(U1-THRES) -> Net-(U1-DISCH)
- R4 pad 1: Net-(Q1-S) -> Net-(U1-DISCH)
- R4 pad 2: Net-(Q1-G) -> Net-(U1-THRES)
- R5 pad 1: Net-(D2-K) -> VCC
- R5 pad 2: GND -> Net-(Q1-G)
- RV1 pad 1: Net-(Q1-S) -> VCC
- SW1 pad 1: /Feeder+ -> Net-(SW1-A)
- SW1 pad 2: /PWM_OUT -> VCC
- SW2 pad 1: Net-(SW2-A) -> /Feeder-
- SW2 pad 2: Net-(Q1-S) -> /PWM_OUT
- U1 pad 4: Net-(Q1-S) -> VCC
- U1 pad 8: Net-(Q1-S) -> VCC
- U2 pad 5: unconnected-(U2B-+-Pad5) -> GND
- U2 pad 6: unconnected-(U2B---Pad6) -> GND
- U2 pad 8: +12V -> VCC
Routing:
- net VCC: track 0.00 -> 92.6 mm
- net +12V: track 0.00 -> 69.5 mm
- net Net-(U2A-+): track 0.00 -> 31.8 mm, vias 0 -> 1
- net Net-(SW1-A): track 0.00 -> 27.5 mm
- net /Feeder+: track 0.00 -> 26.1 mm
- net /Feeder-: track 0.00 -> 25.8 mm
- net Net-(U1-THRES): track 0.00 -> 23.8 mm, vias 0 -> 2
- net /PWM_OUT: track 0.00 -> 12.4 mm
- net Net-(Q1-G): track 0.00 -> 9.19 mm
- net Net-(U1-DISCH): track 0.00 -> 5.85 mm
- net Net-(D1-K): track 0.00 -> 5.80 mm
- net Net-(D2-K): track 0.00 -> 5.80 mm
- added copper zone on B.Cu, net GND
- added copper zone on F.Cu, net GND
Other:
- board outline added: 70 x 70 mm
- board text added: "12V"
- board text added: "1:150 SCALE POWER PACK Designed by @Yu_san_T_robo"
- board text added: "SHORT"
