File: PoweUnit/PoweUnit.kicad_sch (KiCad schematic)
At the start: 1 part, among them U1 NE555D

Commit message: PU回路図書いた
Parts:
- added C1: 0.01u, Capacitor_THT:C_Disc_D5.1mm_W3.2mm_P5.00mm, symbol Device:C
- added C2: 1u, Capacitor_THT:C_Disc_D5.1mm_W3.2mm_P5.00mm, symbol Device:C
- added D1: short, LED_THT:LED_D5.0mm, symbol Device:LED
- added D2: LED, LED_THT:LED_D5.0mm, symbol Device:LED
- added F1: Polyfuse, Fuse:Fuse_Bourns_MF-RG1000, symbol Device:Polyfuse
- added J1: Jack-DC, MyLibrary:MJ-179PH, symbol Connector:Jack-DC
- added J3: Conn_01x02, Connector_JST:JST_XH_S2B-XH-A_1x02_P2.50mm_Horizontal, symbol Connector_Generic:Conn_01x02
- added Q1: Q_PMOS_GDS, Package_TO_SOT_THT:TO-251-3_Vertical, symbol Transistor_FET:Q_PMOS_GDS
- added R1: 5.1k, Resistor_THT:R_Axial_DIN0207_L6.3mm_D2.5mm_P7.62mm_Horizontal, symbol Device:R
- added R2: 1.2k, Resistor_THT:R_Axial_DIN0207_L6.3mm_D2.5mm_P7.62mm_Horizontal, symbol Device:R
- added R3: 3k, Resistor_THT:R_Axial_DIN0207_L6.3mm_D2.5mm_P7.62mm_Horizontal, symbol Device:R
- added R4, R5: 10k, Resistor_THT:R_Axial_DIN0207_L6.3mm_D2.5mm_P7.62mm_Horizontal, symbol Device:R
- added RV1: 10k, samacsys:SL4515NB103L15CM, symbol Device:R_Potentiometer
- added SW1: SW_Slide_DPDT, samacsys:SS22F06G5G, symbol Switch:SW_Slide_DPDT
- added SW2: SW_SPST, MyLibrary:CW-SB11KKFF, symbol Switch:SW_SPST
- added U2: NJM2746M, samacsys:SOIC127P680X200-8N, symbol Device:Opamp_Dual
Connections:
- net GND: now reaches U1.1 (GND)
- net GND: now also C1.2, C2.2, J1.2, R5.2, RV1.3, SW1.5 (B), U2.4 (V-)
- net at U1.2 (TRIG): now also U1.6 (THRES), C1.1, R3.2, U2.2 (-)
- net at U1.4 (~{RST}): now also U1.8 (VCC), C2.1, Q1.3 (S), R2.1, R4.1, RV1.1, SW2.2 (B)
- net at U1.7 (DISCH): now also R2.2, R3.1
- new net: D2.1 (K), R5.1
- new net: F1.2, R1.1, SW2.1 (A)
- new net: Q1.1 (G), R4.2, U2.1
- new net: D1.1 (K), R1.2
- new net: RV1.2, U2.3 (+)
- new net +12V: D1.2 (A), D2.2 (A), F1.1, J1.1, U2.8 (V+)
- new net Feeder+: J3.1 (Pin_1), SW1.1 (A), SW1.4 (A)
- new net Feeder-: J3.2 (Pin_2), SW1.3 (C), SW1.6 (C)
- new net PWM_OUT: Q1.2 (D), SW1.2 (B)
- no-connect marks 0 -> 2
Other:
- note added: "https://akizukidenshi.com/catalog/g/g106568/"
- note added: "https://akizukidenshi.com/catalog/g/g116096/"
- note added: "https://akizukidenshi.com/catalog/g/g117429/"
- note added: "https://akizukidenshi.com/catalog/g/g131326/"
- moved on the sheet: U1

Commit message: パワーパック完成
Parts:
- added C3: 0.1u, Capacitor_THT:C_Disc_D5.1mm_W3.2mm_P5.00mm, symbol Device:C
- added J2: Conn_01x02_Pin, Connector_PinHeader_2.54mm:PinHeader_1x02_P2.54mm_Horizontal, symbol Connector:Conn_01x02_Pin
- added J3: Conn_01x02_Socket, Connector_PinSocket_2.54mm:PinSocket_1x02_P2.54mm_Horizontal, symbol Connector:Conn_01x02_Socket
- added R6: 10k, Resistor_THT:R_Axial_DIN0207_L6.3mm_D2.5mm_P7.62mm_Horizontal, symbol Device:R
- R1: renamed from R5; value 10k -> 5.1k
- renumbered D2 to D1, D1 to D2, J3 to J4, R1 to R2, R2 to R3, R3 to R4, R4 to R5, SW2 to SW1, SW1 to SW2
Connections:
- net +12V: now also J2.1 (Pin_1), J3.1 (Pin_1); no longer U2.8 (V+)
- net Feeder+: now also SW2.3 (C), SW2.6 (C); no longer SW2.1 (A), SW2.4 (A)
- net Feeder-: now also SW2.1 (A), SW2.4 (A); no longer SW2.3 (C), SW2.6 (C)
- net GND: now also U2.5 (+), U2.6 (-), C3.2, J2.2 (Pin_2), J3.2 (Pin_2), R6.2
- net PWM_OUT: now also R6.1
- net VCC: now reaches C2.1, Q1.3 (S), R3.1, R5.1, RV1.1, SW1.2 (B), U1.4 (~{RST}), U1.8 (VCC)
- net VCC: now also U2.8 (V+), C3.1
- no-connect marks 2 -> 3
Other:
- note added: "ACアダプタ"
- note added: "DCジャック"
- note added: "DPDT"
- note added: "PMOS"
- note added: "PWM生成"
- note added: "フィーダ出力"
- note added: "ロッカースイッチ"
- note added: "並列接続用コネクタ"
- note added: "注意 0.5A MAX"
- note removed: "https://akizukidenshi.com/catalog/g/g106568/"
- note removed: "https://akizukidenshi.com/catalog/g/g116096/"
- note removed: "https://akizukidenshi.com/catalog/g/g117429/"
- note removed: "https://akizukidenshi.com/catalog/g/g131326/"
- moved on the sheet: C1, C2, F1, J1, J4, Q1, R1, R2, R3, R4, R5, RV1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
