File: relay-interlocking-machine/relay-interlocking-machine.kicad_sch (KiCad schematic)
At the start: 0 parts

Commit message: リレー論理回路で悩み中
Parts:
- added C1: C, symbol Device:C
- added C2: 1000u, symbol Device:C
- added K1, K6, K7: G5V-2, Relay_THT:Relay_DPDT_Omron_G5V-2, symbol Relay:G5V-2
- added K2, K3, K4, K5: Fujitsu_FTR-LYCA005x, Relay_THT:Relay_SPDT_Fujitsu_FTR-LYCA005x_FormC_Vertical, symbol Relay:Fujitsu_FTR-LYCA005x
- added Q1: NMOS, symbol Transistor_FET_Other:Q_NMOS_Depletion_GDS
- added R1: 10k, symbol Device:R
- added SW1: SW_Rotary_1x4_MP, symbol Switch:SW_Rotary_1x4_MP
- added SW2: PB_A, symbol Switch:SW_SPST
- added SW3, SW5: LV_1, symbol Switch:SW_SPST
- added SW4: PB_B, symbol Switch:SW_SPST
- added U1: 4070, symbol 4xxx:4070
- added U2: 74HC08, symbol MysymbolLibrary:74HC08
Connections:
- new net: C1.1, K4.11
- new net: K2.14, K3.12
- new net: K2.12, K3.14
- new net: U1.3, U2.2
- new net: K6.9, SW2.2 (B), SW3.1 (A)
- new net: K6.16, SW3.2 (B)
- new net: C2.1, K5.11
- new net: K7.9, SW4.2 (B), SW5.1 (A)
- new net: K7.16, SW5.2 (B)
- new net +12V: K2.11, K4.14, K5.14, K6.13, K6.4, K7.13, K7.4, SW2.1 (A), SW4.1 (A)
- new net +3.3V: SW1.1
- new net 51i: K3.11, K4.A1, K5.A1, Q1.1 (G), R1.1, U2.3
- new net FEEDER_51iT_1: K1.6, K1.9
- new net FEEDER_51iT_2: K1.11, K1.8
- new net GND: K1.1, K2.A1, K3.A2, K4.12, K4.A2, K5.12, K5.A2, K6.1, K7.1, Q1.3 (S), R1.2, SW1.2
- new net LV_1: K1.16, SW1.5, U2.1
- new net PB_A: K2.A2, K6.8, U1.1
- new net PB_B: K3.A1, K7.8, U1.2
- new net POINT1: C1.2, C2.2
- new net PWM+: K1.13
- new net PWM-: K1.4, Q1.2 (D)
- no-connect marks 0 -> 7
Other:
- note added: "PWM方向切替"
- note added: "・LVを0にしたときにPBの状態リセット ・PBはモーメンタリで自己保持回路 ・排他的論理和←ではなさそう，1,1を規定してはいけない やりたいこととしては，最後の転轍機を動かすリレーの励磁コイルの01を，PBA,Bと紐づけたい そのうえで，LV1とのANDをとる(=LVを0にしたときにPBの状態リセット)"
- note added: "転轍機操作"
